File: O2_Sensor_Hardware/O2_Sensor_Hardware/O2_Sensor_Hardware.sch (KiCad schematic (older format))
At the start: 2 parts, among them U1 O2_sensor

Commit message: Added Gerbs
Parts:
- U1: symbol O2_Sensor:O2_sensor -> O2_Sensor_Hardware-rescue:O2_sensor-O2_Sensor
Changed lines of the file:
@@
 EESchema Schematic File Version 4
+LIBS:O2_Sensor_Hardware-cache
 EELAYER 30 0
 EELAYER END
@@
 Tx
 $Comp
-L O2_Sensor:O2_sensor U1
+L O2_Sensor_Hardware-rescue:O2_sensor-O2_Sensor U1
 U 1 1 5E72A5E9
 P 1550 1400
